File: hardware/DS8500-test-pcb/DS8500.sch (KiCad schematic (older format))
At the start: 1 part

Commit message: First revision of the DS8500 schematic
Parts:
- added C? (x2): 22p, symbol C_Small
- added C? (x5): 100n, symbol C_Small
- added C? (x2): 1u, symbol C_Small
- added JP? (x3): Jumper_NO_Small, symbol Jumper_NO_Small
- added P?: CONN_01X03, symbol CONN_01X03
- added P?: CONN_01X02, symbol CONN_01X02
- added R? (x2): 20k, symbol R_Small
- added R? (x2): 10k, symbol R_Small
- added U?: AP1117V5, symbol AP1117
- added W?: FSK_OUT, symbol TEST_1P
- added W?: GND, symbol TEST_1P
- added Y?: 3.6864MHz, symbol Crystal_Small
Connections:
- net labels added: +5V, GND, VCC
- wire segments 0 -> 70
- no-connect marks 0 -> 4
Other:
- moved on the sheet: U?
