File: hardware/DS8500-test-pcb/DS8500.sch (KiCad schematic (older format))
At the start: 23 parts, among them P1 POWER, P2 INTERFACE, U1 AP1117V5, U2 DS8500, Y1 3.6864MHz

Commit message: Added extra test points at the input
Parts:
- added W3: FSK_IN, Pin_Headers:Pin_Header_Straight_1x01, symbol TEST_1P
- added W4: GND, Pin_Headers:Pin_Header_Straight_1x01, symbol TEST_1P
Connections:
- wire segments 70 -> 71
Changed lines of the file:
@@
 LIBS:conn_16_mirror
 LIBS:conn_16
+LIBS:DS8500-cache
 EELAYER 25 0
 EELAYER END
@@
 	3550 3300 5400 3300
 Wire Wire Line
-	3650 3300 3650 3450
+	3650 3200 3650 3450
 Wire Wire Line
 	4200 3750 4200 3700
@@
 	7050 4050 7050 4100
 Connection ~ 6800 4050
+$Comp
+L TEST_1P W3
+U 1 1 572345F3
+P 3650 3200
+F 0 "W3" H 3650 3470 50  0000 C CNN
+F 1 "FSK_IN" H 3650 3400 50  0000 C CNN
+F 2 "Pin_Headers:Pin_Header_Straight_1x01" H 3850 3200 50  0001 C CNN
+F 3 "" H 3850 3200 50  0000 C CNN
+	1    3650 3200
+	1    0    0    -1
+$EndComp
+$Comp
+L TEST_1P W4
+U 1 1 57234BE3
+P 3650 4350
+F 0 "W4" H 3650 4620 50  0000 C CNN
+F 1 "GND" H 3650 4550 50  0000 C CNN
+F 2 "Pin_Headers:Pin_Header_Straight_1x01" H 3850 4350 50  0001 C CNN
+F 3 "" H 3850 4350 50  0000 C CNN
+	1    3650 4350
+	1    0    0    -1
+$EndComp
+$Comp
+L GND #PWR019
+U 1 1 57234C50
+P 3650 4450
+F 0 "#PWR019" H 3650 4200 50  0001 C CNN
+F 1 "GND" H 3650 4300 50  0000 C CNN
+F 2 "" H 3650 4450 50  0000 C CNN
+F 3 "" H 3650 4450 50  0000 C CNN
+	1    3650 4450
+	1    0    0    -1
+$EndComp
+Wire Wire Line
+	3650 4450 3650 4350
 $EndSCHEMATC

Commit message: No need for RTS. We will be always in MODULATOR mode -> RTS pin tied to GND
Parts:
- removed JP1, JP2: Jumper_NO_Small, Pin_Headers:Pin_Header_Straight_1x02, symbol Jumper_NO_Small
- removed P2: INTERFACE, Pin_Headers:Pin_Header_Straight_1x03, symbol CONN_01X03
- removed R1: 10k, w_smd_resistors:r_0805, symbol R_Small
- removed R2: 20k, w_smd_resistors:r_0805, symbol R_Small
- added P2: INTERFACE, Pin_Headers:Pin_Header_Straight_1x02, symbol CONN_01X02
Connections:
- wire segments 71 -> 65
Other:
- moved on the sheet: W3
Changed lines of the file:
@@
 $EndComp
 $Comp
-L GND #PWR01
+L GND #PWR13
 U 1 1 571F7D34
 P 5950 4600
-F 0 "#PWR01" H 5950 4350 50  0001 C CNN
+F 0 "#PWR13" H 5950 4350 50  0001 C CNN
 F 1 "GND" H 5950 4450 50  0000 C CNN
 F 2 "" H 5950 4600 50  0000 C CNN
@@
 $EndComp
 $Comp
-L VCC #PWR02
+L VCC #PWR12
 U 1 1 571F7ECB
 P 5950 2100
-F 0 "#PWR02" H 5950 1950 50  0001 C CNN
+F 0 "#PWR12" H 5950 1950 50  0001 C CNN
 F 1 "VCC" H 5950 2250 50  0000 C CNN
 F 2 "" H 5950 2100 50  0000 C CNN
@@
 $EndComp
 $Comp
-L GND #PWR03
+L GND #PWR9
 U 1 1 571F83A1
 P 4250 2800
-F 0 "#PWR03" H 4250 2550 50  0001 C CNN
+F 0 "#PWR9" H 4250 2550 50  0001 C CNN
 F 1 "GND" H 4250 2650 50  0000 C CNN
 F 2 "" H 4250 2800 50  0000 C CNN
@@
 $EndComp
 $Comp
-L GND #PWR04
+L GND #PWR11
 U 1 1 571F862F
 P 5150 3000
-F 0 "#PWR04" H 5150 2750 50  0001 C CNN
+F 0 "#PWR11" H 5150 2750 50  0001 C CNN
 F 1 "GND" H 5150 2850 50  0000 C CNN
 F 2 "" H 5150 3000 50  0000 C CNN
@@
 $EndComp
 $Comp
-L GND #PWR05
+L GND #PWR16
 U 1 1 571F877B
 P 6850 3000
-F 0 "#PWR05" H 6850 2750 50  0001 C CNN
+F 0 "#PWR16" H 6850 2750 50  0001 C CNN
 F 1 "GND" H 6850 2850 50  0000 C CNN
 F 2 "" H 6850 3000 50  0000 C CNN
@@
 NoConn ~ 5400 3850
 $Comp
-L VCC #PWR06
+L VCC #PWR10
 U 1 1 571F88B0
-P 5250 3600
-F 0 "#PWR06" H 5250 3450 50  0001 C CNN
-F 1 "VCC" H 5250 3750 50  0000 C CNN
-F 2 "" H 5250 3600 50  0000 C CNN
-F 3 "" H 5250 3600 50  0000 C CNN
-	1    5250 3600
+P 5100 3600
+F 0 "#PWR10" H 5100 3450 50  0001 C CNN
+F 1 "VCC" H 5100 3750 50  0000 C CNN
+F 2 "" H 5100 3600 50  0000 C CNN
+F 3 "" H 5100 3600 50  0000 C CNN
+	1    5100 3600
 	1    0    0    -1
 $EndComp
@@
 $EndComp
 $Comp
-L GND #PWR07
+L GND #PWR17
 U 1 1 571F946D
 P 7650 4100
-F 0 "#PWR07" H 7650 3850 50  0001 C CNN
+F 0 "#PWR17" H 7650 3850 50  0001 C CNN
 F 1 "GND" H 7650 3950 50  0000 C CNN
 F 2 "" H 7650 4100 50  0000 C CNN
 F 3 "" H 7650 4100 50  0000 C CNN
 	1    7650 4100
-	1    0    0    -1
-$EndComp
-$Comp
-L CONN_01X03 P2
-U 1 1 571F97AB
-P 2900 3400
-F 0 "P2" H 2900 3600 50  0000 C CNN
-F 1 "INTERFACE" V 3000 3400 50  0000 C CNN
-F 2 "Pin_Headers:Pin_Header_Straight_1x03" H 2900 3400 50  0001 C CNN
-F 3 "" H 2900 3400 50  0000 C CNN
-	1    2900 3400
-	-1   0    0    1
-$EndComp
-$Comp
-L Jumper_NO_Small JP1
-U 1 1 571F99DD
-P 4650 3650
-F 0 "JP1" H 4650 3730 50  0000 C CNN
-F 1 "Jumper_NO_Small" H 4660 3590 50  0001 C CNN
-F 2 "Pin_Headers:Pin_Header_Straight_1x02" H 4650 3650 50  0001 C CNN
-F 3 "" H 4650 3650 50  0000 C CNN
-	1    4650 3650
-	1    0    0    -1
-$EndComp
-$Comp
-L Jumper_NO_Small JP2
-U 1 1 571F9A44
-P 4950 3650
-F 0 "JP2" H 4950 3730 50  0000 C CNN
-F 1 "Jumper_NO_Small" H 4960 3590 50  0001 C CNN
-F 2 "Pin_Headers:Pin_Header_Straight_1x02" H 4950 3650 50  0001 C CNN
-F 3 "" H 4950 3650 50  0000 C CNN
-	1    4950 3650
-	1    0    0    -1
-$EndComp
-$Comp
-L R_Small R2
-U 1 1 571FA000
-P 3650 3550
-F 0 "R2" H 3680 3570 50  0000 L CNN
-F 1 "20k" H 3680 3510 50  0000 L CNN
-F 2 "w_smd_resistors:r_0805" H 3650 3550 50  0001 C CNN
-F 3 "" H 3650 3550 50  0000 C CNN
-	1    3650 3550
-	1    0    0    -1
-$EndComp
-$Comp
-L R_Small R1
-U 1 1 571FA07B
-P 3450 3300
-F 0 "R1" V 3500 3400 50  0000 L CNN
-F 1 "10k" V 3550 3150 50  0000 L CNN
-F 2 "w_smd_resistors:r_0805" H 3450 3300 50  0001 C CNN
-F 3 "" H 3450 3300 50  0000 C CNN
-	1    3450 3300
-	0    -1   -1   0
-$EndComp
-$Comp
-L GND #PWR08
-U 1 1 571FA0BF
-P 3650 3700
-F 0 "#PWR08" H 3650 3450 50  0001 C CNN
-F 1 "GND" H 3650 3550 50  0000 C CNN
-F 2 "" H 3650 3700 50  0000 C CNN
-F 3 "" H 3650 3700 50  0000 C CNN
-	1    3650 3700
 	1    0    0    -1
 $EndComp
@@
 $EndComp
 $Comp
-L GND #PWR09
+L GND #PWR8
 U 1 1 571FA3C1
 P 4200 3750
-F 0 "#PWR09" H 4200 3500 50  0001 C CNN
+F 0 "#PWR8" H 4200 3500 50  0001 C CNN
 F 1 "GND" H 4200 3600 50  0000 C CNN
 F 2 "" H 4200 3750 50  0000 C CNN
@@
 $EndComp
 $Comp
-L GND #PWR010
-U 1 1 571FA6F2
-P 4500 3900
-F 0 "#PWR010" H 4500 3650 50  0001 C CNN
-F 1 "GND" H 4500 3750 50  0000 C CNN
-F 2 "" H 4500 3900 50  0000 C CNN
-F 3 "" H 4500 3900 50  0000 C CNN
-	1    4500 3900
-	1    0    0    -1
-$EndComp
-$Comp
-L GND #PWR011
+L GND #PWR3
 U 1 1 571FB69A
 P 3200 3550
-F 0 "#PWR011" H 3200 3300 50  0001 C CNN
+F 0 "#PWR3" H 3200 3300 50  0001 C CNN
 F 1 "GND" H 3200 3400 50  0000 C CNN
 F 2 "" H 3200 3550 50  0000 C CNN
@@
 $EndComp
 $Comp
-L GND #PWR012
+L GND #PWR2
 U 1 1 571FB87A
 P 3200 2950
-F 0 "#PWR012" H 3200 2700 50  0001 C CNN
+F 0 "#PWR2" H 3200 2700 50  0001 C CNN
 F 1 "GND" H 3200 2800 50  0000 C CNN
 F 2 "" H 3200 2950 50  0000 C CNN
@@
 $EndComp
 $Comp
-L +5V #PWR013
+L +5V #PWR1
 U 1 1 571FB9EE
 P 3200 2650
-F 0 "#PWR013" H 3200 2500 50  0001 C CNN
+F 0 "#PWR1" H 3200 2500 50  0001 C CNN
 F 1 "+5V" H 3200 2790 50  0000 C CNN
 F 2 "" H 3200 2650 50  0000 C CNN
@@
 $EndComp
 $Comp
-L VCC #PWR014
+L VCC #PWR7
 U 1 1 571FBE79
 P 4200 1700
-F 0 "#PWR014" H 4200 1550 50  0001 C CNN
+F 0 "#PWR7" H 4200 1550 50  0001 C CNN
 F 1 "VCC" H 4200 1850 50  0000 C CNN
 F 2 "" H 4200 1700 50  0000 C CNN
@@
 $EndComp
 $Comp
-L +5V #PWR015
+L +5V #PWR4
 U 1 1 571FBF1F
 P 3400 1700
-F 0 "#PWR015" H 3400 1550 50  0001 C CNN
+F 0 "#PWR4" H 3400 1550 50  0001 C CNN
 F 1 "+5V" H 3400 1840 50  0000 C CNN
 F 2 "" H 3400 1700 50  0000 C CNN
@@
 $EndComp
 $Comp
-L GND #PWR016
+L GND #PWR6
 U 1 1 571FBFAF
 P 3800 2200
-F 0 "#PWR016" H 3800 1950 50  0001 C CNN
+F 0 "#PWR6" H 3800 1950 50  0001 C CNN
 F 1 "GND" H 3800 2050 50  0000 C CNN
 F 2 "" H 3800 2200 50  0000 C CNN
@@
 $EndComp
 $Comp
-L GND #PWR017
+L GND #PWR15
 U 1 1 571FD283
 P 6800 4500
-F 0 "#PWR017" H 6800 4250 50  0001 C CNN
+F 0 "#PWR15" H 6800 4250 50  0001 C CNN
 F 1 "GND" H 6800 4350 50  0000 C CNN
 F 2 "" H 6800 4500 50  0000 C CNN
@@
 	6850 3000 6750 3000
 Wire Wire Line
-	5250 3600 5250 3650
-Wire Wire Line
-	5050 3650 5400 3650
-Wire Wire Line
 	6500 3350 7400 3350
 Wire Wire Line
@@
 Wire Wire Line
 	7650 4000 7800 4000
-Wire Wire Line
-	4750 3650 4850 3650
-Wire Wire Line
-	4800 3300 4800 3650
-Connection ~ 4800 3300
-Connection ~ 4800 3650
 Connection ~ 5250 3650
 Wire Wire Line
-	3650 3700 3650 3650
-Wire Wire Line
-	3550 3300 5400 3300
-Wire Wire Line
-	3650 3200 3650 3450
-Wire Wire Line
 	4200 3750 4200 3700
 Wire Wire Line
 	4100 3400 5400 3400
 Wire Wire Line
-	4200 3400 4200 3500
-Wire Wire Line
-	4500 3900 4500 3650
-Wire Wire Line
-	4500 3650 4550 3650
+	4200 3350 4200 3500
 Connection ~ 4200 3400
-Connection ~ 3650 3300
-Wire Wire Line
-	3100 3300 3350 3300
 Wire Wire Line
 	3100 3400 3900 3400
@@
 Connection ~ 6800 4400
 $Comp
-L VCC #PWR018
+L VCC #PWR14
 U 1 1 571FD437
 P 6800 4000
-F 0 "#PWR018" H 6800 3850 50  0001 C CNN
+F 0 "#PWR14" H 6800 3850 50  0001 C CNN
 F 1 "VCC" H 6800 4150 50  0000 C CNN
 F 2 "" H 6800 4000 50  0000 C CNN
@@
 L TEST_1P W3
 U 1 1 572345F3
-P 3650 3200
-F 0 "W3" H 3650 3470 50  0000 C CNN
-F 1 "FSK_IN" H 3650 3400 50  0000 C CNN
-F 2 "Pin_Headers:Pin_Header_Straight_1x01" H 3850 3200 50  0001 C CNN
-F 3 "" H 3850 3200 50  0000 C CNN
-	1    3650 3200
+P 4200 3350
+F 0 "W3" H 4200 3620 50  0000 C CNN
+F 1 "FSK_IN" H 4200 3550 50  0000 C CNN
+F 2 "Pin_Headers:Pin_Header_Straight_1x01" H 4400 3350 50  0001 C CNN
+F 3 "" H 4400 3350 50  0000 C CNN
+	1    4200 3350
 	1    0    0    -1
 $EndComp
@@
 $EndComp
 $Comp
-L GND #PWR019
+L GND #PWR5
 U 1 1 57234C50
 P 3650 4450
-F 0 "#PWR019" H 3650 4200 50  0001 C CNN
+F 0 "#PWR5" H 3650 4200 50  0001 C CNN
 F 1 "GND" H 3650 4300 50  0000 C CNN
 F 2 "" H 3650 4450 50  0000 C CNN
@@
 Wire Wire Line
 	3650 4450 3650 4350
+Wire Wire Line
+	5100 3650 5400 3650
+Wire Wire Line
+	5100 3600 5100 3650
+$Comp
+L CONN_01X02 P2
+U 1 1 5723CD7B
+P 2900 3450
+F 0 "P2" H 2900 3600 50  0000 C CNN
+F 1 "INTERFACE" V 3000 3450 50  0000 C CNN
+F 2 "Pin_Headers:Pin_Header_Straight_1x02" H 2900 3450 50  0001 C CNN
+F 3 "" H 2900 3450 50  0000 C CNN
+	1    2900 3450
+	-1   0    0    1
+$EndComp
+Wire Wire Line
+	5400 3300 5300 3300
+Wire Wire Line
+	5300 3300 5300 2950
+Connection ~ 5300 2950
 $EndSCHEMATC

Commit message: 0-OHM jumper resistor
Parts:
- added R1: 0, symbol R_Small
Connections:
- net at R3.2, R4.1, W3.1: now also R1.1; no longer U2.20 (D_IN)
- new net: R1.2, U2.20 (D_IN)
Changed lines of the file:
@@
 	1    0    0    -1
 $EndComp
-Wire Wire Line
-	5950 4400 5950 4600
-Wire Wire Line
-	5750 4500 6150 4500
-Wire Wire Line
-	5750 4500 5750 4400
-Wire Wire Line
-	6150 4500 6150 4400
-Connection ~ 5950 4500
-Wire Wire Line
-	6050 4400 6050 4500
-Connection ~ 6050 4500
-Wire Wire Line
-	5850 4500 5850 4400
-Connection ~ 5850 4500
-Wire Wire Line
-	5950 2100 5950 2300
-Wire Wire Line
-	5850 2200 6050 2200
-Wire Wire Line
-	5850 2200 5850 2300
-Wire Wire Line
-	6050 2200 6050 2300
-Connection ~ 5950 2200
-Wire Wire Line
-	4850 2700 4850 2650
-Wire Wire Line
-	4600 2650 5050 2650
-Wire Wire Line
-	5050 2650 5050 2750
-Wire Wire Line
-	5050 2750 5400 2750
-Wire Wire Line
-	5400 2850 5050 2850
-Wire Wire Line
-	5050 2850 5050 2950
-Wire Wire Line
-	5050 2950 4600 2950
-Wire Wire Line
-	4850 2950 4850 2900
-Connection ~ 4850 2650
-Connection ~ 4850 2950
-Wire Wire Line
-	4250 2800 4300 2800
-Wire Wire Line
-	4300 2650 4300 2950
-Wire Wire Line
-	4300 2650 4400 2650
-Wire Wire Line
-	4300 2950 4400 2950
-Connection ~ 4300 2800
-Wire Wire Line
-	5400 2950 5150 2950
-Wire Wire Line
-	5150 2950 5150 3000
-Wire Wire Line
-	6550 3000 6500 3000
-Wire Wire Line
-	6850 3000 6750 3000
-Wire Wire Line
-	6500 3350 7400 3350
-Wire Wire Line
-	7400 3200 7300 3200
-Wire Wire Line
-	7300 3200 7300 3650
-Connection ~ 7300 3350
-Wire Wire Line
-	7600 3200 7700 3200
-Wire Wire Line
-	7700 3200 7700 3650
-Wire Wire Line
-	7600 3350 7800 3350
-Connection ~ 7700 3350
-Wire Wire Line
-	7300 3650 7400 3650
-Wire Wire Line
-	7700 3650 7600 3650
-Wire Wire Line
-	7650 4100 7650 4000
-Wire Wire Line
-	7650 4000 7800 4000
-Connection ~ 5250 3650
-Wire Wire Line
-	4200 3750 4200 3700
-Wire Wire Line
-	4100 3400 5400 3400
-Wire Wire Line
-	4200 3350 4200 3500
-Connection ~ 4200 3400
-Wire Wire Line
-	3100 3400 3900 3400
-Wire Wire Line
-	3200 3550 3200 3500
-Wire Wire Line
-	3200 3500 3100 3500
-Wire Wire Line
-	3200 2950 3200 2850
-Wire Wire Line
-	3200 2850 3100 2850
-Wire Wire Line
-	3200 2650 3200 2750
-Wire Wire Line
-	3200 2750 3100 2750
-Wire Wire Line
-	4200 1700 4200 1900
-Wire Wire Line
-	4200 1800 4100 1800
-Wire Wire Line
-	3400 1700 3400 1900
-Wire Wire Line
-	3400 1800 3500 1800
-Wire Wire Line
-	3800 2200 3800 2100
-Connection ~ 3400 1800
-Wire Wire Line
-	3400 2100 3400 2150
-Wire Wire Line
-	3400 2150 4200 2150
-Connection ~ 3800 2150
-Wire Wire Line
-	4200 2150 4200 2100
-Connection ~ 4200 1800
-Wire Wire Line
-	6800 4500 6800 4300
-Wire Wire Line
-	7050 4300 7050 4400
-Wire Wire Line
-	7050 4400 6800 4400
-Connection ~ 6800 4400
 $Comp
 L VCC #PWR14
@@
 	1    0    0    -1
 $EndComp
-Wire Wire Line
-	6800 4000 6800 4100
-Wire Wire Line
-	6800 4050 7050 4050
-Wire Wire Line
-	7050 4050 7050 4100
-Connection ~ 6800 4050
 $Comp
 L TEST_1P W3
@@
 	1    0    0    -1
 $EndComp
-Wire Wire Line
-	3650 4450 3650 4350
-Wire Wire Line
-	5100 3650 5400 3650
-Wire Wire Line
-	5100 3600 5100 3650
 $Comp
 L CONN_01X02 P2
@@
 	-1   0    0    1
 $EndComp
+$Comp
+L R_Small R1
+U 1 1 5723DA3F
+P 4650 3400
+F 0 "R1" H 4680 3420 50  0000 L CNN
+F 1 "0" H 4680 3360 50  0000 L CNN
+F 2 "" H 4650 3400 50  0000 C CNN
+F 3 "" H 4650 3400 50  0000 C CNN
+	1    4650 3400
+	0    -1   -1   0
+$EndComp
+Wire Wire Line
+	5950 4400 5950 4600
+Wire Wire Line
+	5750 4500 6150 4500
+Wire Wire Line
+	5750 4500 5750 4400
+Wire Wire Line
+	6150 4500 6150 4400
+Connection ~ 5950 4500
+Wire Wire Line
+	6050 4400 6050 4500
+Connection ~ 6050 4500
+Wire Wire Line
+	5850 4500 5850 4400
+Connection ~ 5850 4500
+Wire Wire Line
+	5950 2100 5950 2300
+Wire Wire Line
+	5850 2200 6050 2200
+Wire Wire Line
+	5850 2200 5850 2300
+Wire Wire Line
+	6050 2200 6050 2300
+Connection ~ 5950 2200
+Wire Wire Line
+	4850 2700 4850 2650
+Wire Wire Line
+	4600 2650 5050 2650
+Wire Wire Line
+	5050 2650 5050 2750
+Wire Wire Line
+	5050 2750 5400 2750
+Wire Wire Line
+	5400 2850 5050 2850
+Wire Wire Line
+	5050 2850 5050 2950
+Wire Wire Line
+	5050 2950 4600 2950
+Wire Wire Line
+	4850 2950 4850 2900
+Connection ~ 4850 2650
+Connection ~ 4850 2950
+Wire Wire Line
+	4250 2800 4300 2800
+Wire Wire Line
+	4300 2650 4300 2950
+Wire Wire Line
+	4300 2650 4400 2650
+Wire Wire Line
+	4300 2950 4400 2950
+Connection ~ 4300 2800
+Wire Wire Line
+	5400 2950 5150 2950
+Wire Wire Line
+	5150 2950 5150 3000
+Wire Wire Line
+	6550 3000 6500 3000
+Wire Wire Line
+	6850 3000 6750 3000
+Wire Wire Line
+	6500 3350 7400 3350
+Wire Wire Line
+	7400 3200 7300 3200
+Wire Wire Line
+	7300 3200 7300 3650
+Connection ~ 7300 3350
+Wire Wire Line
+	7600 3200 7700 3200
+Wire Wire Line
+	7700 3200 7700 3650
+Wire Wire Line
+	7600 3350 7800 3350
+Connection ~ 7700 3350
+Wire Wire Line
+	7300 3650 7400 3650
+Wire Wire Line
+	7700 3650 7600 3650
+Wire Wire Line
+	7650 4100 7650 4000
+Wire Wire Line
+	7650 4000 7800 4000
+Connection ~ 5250 3650
+Wire Wire Line
+	4200 3750 4200 3700
+Wire Wire Line
+	4200 3350 4200 3500
+Connection ~ 4200 3400
+Wire Wire Line
+	3100 3400 3900 3400
+Wire Wire Line
+	3200 3550 3200 3500
+Wire Wire Line
+	3200 3500 3100 3500
+Wire Wire Line
+	3200 2950 3200 2850
+Wire Wire Line
+	3200 2850 3100 2850
+Wire Wire Line
+	3200 2650 3200 2750
+Wire Wire Line
+	3200 2750 3100 2750
+Wire Wire Line
+	4200 1700 4200 1900
+Wire Wire Line
+	4200 1800 4100 1800
+Wire Wire Line
+	3400 1700 3400 1900
+Wire Wire Line
+	3400 1800 3500 1800
+Wire Wire Line
+	3800 2200 3800 2100
+Connection ~ 3400 1800
+Wire Wire Line
+	3400 2100 3400 2150
+Wire Wire Line
+	3400 2150 4200 2150
+Connection ~ 3800 2150
+Wire Wire Line
+	4200 2150 4200 2100
+Connection ~ 4200 1800
+Wire Wire Line
+	6800 4500 6800 4300
+Wire Wire Line
+	7050 4300 7050 4400
+Wire Wire Line
+	7050 4400 6800 4400
+Connection ~ 6800 4400
+Wire Wire Line
+	6800 4000 6800 4100
+Wire Wire Line
+	6800 4050 7050 4050
+Wire Wire Line
+	7050 4050 7050 4100
+Connection ~ 6800 4050
+Wire Wire Line
+	3650 4450 3650 4350
+Wire Wire Line
+	5100 3650 5400 3650
+Wire Wire Line
+	5100 3600 5100 3650
 Wire Wire Line
 	5400 3300 5300 3300
@@
 	5300 3300 5300 2950
 Connection ~ 5300 2950
+Wire Wire Line
+	4100 3400 4550 3400
+Wire Wire Line
+	4750 3400 5400 3400
 $EndSCHEMATC

Commit message: Beta(?) version of the PCB
Parts:
- R1: footprint (none) -> w_smd_resistors:r_0805
Changed lines of the file:
@@
 $EndComp
 $Comp
-L GND #PWR13
+L GND #PWR01
 U 1 1 571F7D34
 P 5950 4600
-F 0 "#PWR13" H 5950 4350 50  0001 C CNN
+F 0 "#PWR01" H 5950 4350 50  0001 C CNN
 F 1 "GND" H 5950 4450 50  0000 C CNN
 F 2 "" H 5950 4600 50  0000 C CNN
@@
 $EndComp
 $Comp
-L VCC #PWR12
+L VCC #PWR02
 U 1 1 571F7ECB
 P 5950 2100
-F 0 "#PWR12" H 5950 1950 50  0001 C CNN
+F 0 "#PWR02" H 5950 1950 50  0001 C CNN
 F 1 "VCC" H 5950 2250 50  0000 C CNN
 F 2 "" H 5950 2100 50  0000 C CNN
@@
 $EndComp
 $Comp
-L GND #PWR9
+L GND #PWR03
 U 1 1 571F83A1
 P 4250 2800
-F 0 "#PWR9" H 4250 2550 50  0001 C CNN
+F 0 "#PWR03" H 4250 2550 50  0001 C CNN
 F 1 "GND" H 4250 2650 50  0000 C CNN
 F 2 "" H 4250 2800 50  0000 C CNN
@@
 $EndComp
 $Comp
-L GND #PWR11
+L GND #PWR04
 U 1 1 571F862F
 P 5150 3000
-F 0 "#PWR11" H 5150 2750 50  0001 C CNN
+F 0 "#PWR04" H 5150 2750 50  0001 C CNN
 F 1 "GND" H 5150 2850 50  0000 C CNN
 F 2 "" H 5150 3000 50  0000 C CNN
@@
 $EndComp
 $Comp
-L GND #PWR16
+L GND #PWR05
 U 1 1 571F877B
 P 6850 3000
-F 0 "#PWR16" H 6850 2750 50  0001 C CNN
+F 0 "#PWR05" H 6850 2750 50  0001 C CNN
 F 1 "GND" H 6850 2850 50  0000 C CNN
 F 2 "" H 6850 3000 50  0000 C CNN
@@
 NoConn ~ 5400 3850
 $Comp
-L VCC #PWR10
+L VCC #PWR06
 U 1 1 571F88B0
 P 5100 3600
-F 0 "#PWR10" H 5100 3450 50  0001 C CNN
+F 0 "#PWR06" H 5100 3450 50  0001 C CNN
 F 1 "VCC" H 5100 3750 50  0000 C CNN
 F 2 "" H 5100 3600 50  0000 C CNN
@@
 $EndComp
 $Comp
-L GND #PWR17
+L GND #PWR07
 U 1 1 571F946D
 P 7650 4100
-F 0 "#PWR17" H 7650 3850 50  0001 C CNN
+F 0 "#PWR07" H 7650 3850 50  0001 C CNN
 F 1 "GND" H 7650 3950 50  0000 C CNN
 F 2 "" H 7650 4100 50  0000 C CNN
@@
 $EndComp
 $Comp
-L GND #PWR8
+L GND #PWR08
 U 1 1 571FA3C1
 P 4200 3750
-F 0 "#PWR8" H 4200 3500 50  0001 C CNN
+F 0 "#PWR08" H 4200 3500 50  0001 C CNN
 F 1 "GND" H 4200 3600 50  0000 C CNN
 F 2 "" H 4200 3750 50  0000 C CNN
@@
 $EndComp
 $Comp
-L GND #PWR3
+L GND #PWR09
 U 1 1 571FB69A
 P 3200 3550
-F 0 "#PWR3" H 3200 3300 50  0001 C CNN
+F 0 "#PWR09" H 3200 3300 50  0001 C CNN
 F 1 "GND" H 3200 3400 50  0000 C CNN
 F 2 "" H 3200 3550 50  0000 C CNN
@@
 $EndComp
 $Comp
-L GND #PWR2
+L GND #PWR010
 U 1 1 571FB87A
 P 3200 2950
-F 0 "#PWR2" H 3200 2700 50  0001 C CNN
+F 0 "#PWR010" H 3200 2700 50  0001 C CNN
 F 1 "GND" H 3200 2800 50  0000 C CNN
 F 2 "" H 3200 2950 50  0000 C CNN
@@
 $EndComp
 $Comp
-L +5V #PWR1
+L +5V #PWR011
 U 1 1 571FB9EE
 P 3200 2650
-F 0 "#PWR1" H 3200 2500 50  0001 C CNN
+F 0 "#PWR011" H 3200 2500 50  0001 C CNN
 F 1 "+5V" H 3200 2790 50  0000 C CNN
 F 2 "" H 3200 2650 50  0000 C CNN
@@
 $EndComp
 $Comp
-L VCC #PWR7
+L VCC #PWR012
 U 1 1 571FBE79
 P 4200 1700
-F 0 "#PWR7" H 4200 1550 50  0001 C CNN
+F 0 "#PWR012" H 4200 1550 50  0001 C CNN
 F 1 "VCC" H 4200 1850 50  0000 C CNN
 F 2 "" H 4200 1700 50  0000 C CNN
@@
 $EndComp
 $Comp
-L +5V #PWR4
+L +5V #PWR013
 U 1 1 571FBF1F
 P 3400 1700
-F 0 "#PWR4" H 3400 1550 50  0001 C CNN
+F 0 "#PWR013" H 3400 1550 50  0001 C CNN
 F 1 "+5V" H 3400 1840 50  0000 C CNN
 F 2 "" H 3400 1700 50  0000 C CNN
@@
 $EndComp
 $Comp
-L GND #PWR6
+L GND #PWR014
 U 1 1 571FBFAF
 P 3800 2200
-F 0 "#PWR6" H 3800 1950 50  0001 C CNN
+F 0 "#PWR014" H 3800 1950 50  0001 C CNN
 F 1 "GND" H 3800 2050 50  0000 C CNN
 F 2 "" H 3800 2200 50  0000 C CNN
@@
 $EndComp
 $Comp
-L GND #PWR15
+L GND #PWR015
 U 1 1 571FD283
 P 6800 4500
-F 0 "#PWR15" H 6800 4250 50  0001 C CNN
+F 0 "#PWR015" H 6800 4250 50  0001 C CNN
 F 1 "GND" H 6800 4350 50  0000 C CNN
 F 2 "" H 6800 4500 50  0000 C CNN
@@
 $EndComp
 $Comp
-L VCC #PWR14
+L VCC #PWR016
 U 1 1 571FD437
 P 6800 4000
-F 0 "#PWR14" H 6800 3850 50  0001 C CNN
+F 0 "#PWR016" H 6800 3850 50  0001 C CNN
 F 1 "VCC" H 6800 4150 50  0000 C CNN
 F 2 "" H 6800 4000 50  0000 C CNN
@@
 $EndComp
 $Comp
-L GND #PWR5
+L GND #PWR017
 U 1 1 57234C50
 P 3650 4450
-F 0 "#PWR5" H 3650 4200 50  0001 C CNN
+F 0 "#PWR017" H 3650 4200 50  0001 C CNN
 F 1 "GND" H 3650 4300 50  0000 C CNN
 F 2 "" H 3650 4450 50  0000 C CNN
@@
 F 0 "R1" H 4680 3420 50  0000 L CNN
 F 1 "0" H 4680 3360 50  0000 L CNN
-F 2 "" H 4650 3400 50  0000 C CNN
+F 2 "w_smd_resistors:r_0805" H 4650 3400 50  0001 C CNN
 F 3 "" H 4650 3400 50  0000 C CNN
 	1    4650 3400

Commit message: Wrong package for DS8500. The correct one is TQFN-20 5x5mm
Parts:
- U2: footprint w_smd_qfn:qfn-20 -> Housings_DFN_QFN:QFN-20-1EP_5x5mm_Pitch0.65mm
Changed lines of the file:
@@
 F 0 "U2" H 6350 2300 60  0000 C CNN
 F 1 "DS8500" H 6300 4200 60  0000 C CNN
-F 2 "w_smd_qfn:qfn-20" H 5950 3650 60  0001 C CNN
+F 2 "Housings_DFN_QFN:QFN-20-1EP_5x5mm_Pitch0.65mm" H 5950 3650 60  0001 C CNN
 F 3 "" H 5950 3650 60  0000 C CNN
 	1    5950 3300

Commit message: Extended the leads of the TQFN-20 for hand soldering
Parts:
- removed R1: 0, w_smd_resistors:r_0805, symbol R_Small
Connections:
- net at U2.20 (D_IN): now also R3.2, R4.1, W3.1
Changed lines of the file:
@@
 	-1   0    0    1
-$EndComp
-$Comp
-L R_Small R1
-U 1 1 5723DA3F
-P 4650 3400
-F 0 "R1" H 4680 3420 50  0000 L CNN
-F 1 "0" H 4680 3360 50  0000 L CNN
-F 2 "w_smd_resistors:r_0805" H 4650 3400 50  0001 C CNN
-F 3 "" H 4650 3400 50  0000 C CNN
-	1    4650 3400
-	0    -1   -1   0
 $EndComp
 Wire Wire Line
@@
 Connection ~ 5300 2950
 Wire Wire Line
-	4100 3400 4550 3400
-Wire Wire Line
-	4750 3400 5400 3400
+	4100 3400 5400 3400
 $EndSCHEMATC
